File: PD Board/PD Board.kicad_sch (KiCad schematic)
At the start: 19 parts, among them J1 Conn_02x02_Odd_Even, M1 2002411112, P1 2604-1102, P2 2604-1102, P3 2604-1102, P4 2604-1102, P5 2604-1102, P6 2604-1102, P7 2604-1102, P8 2604-1102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

Commit message: moved tab
Parts:
- removed M1: 2002411112, MOLEXMega:CONN_2002411000_02_MOL, symbol 2025-08-04_21-40-05:2002411112
- added P9: 2604-1102, Customconnectors:26041102, symbol 2604-1102:2604-1102
- D1: footprint CustomImports:LTST-C930 -> Customconnectors:LTST-C930
- P1, P2, P3, P4, P5, P6, P7, P8: footprint Capacitor:26041102 -> Customconnectors:26041102
- U1: footprint MCP1792T3302HCB:SOT-23A_CB_MCH -> Customconnectors:SOT-23A_CB_MCH
Connections:
- net +20V: now also P9.3 (2.1), P9.4 (2.2)
- net GND: now also P9.1 (1.1), P9.2 (1.2)
