File: DistanceSensor/DistanceSensor.kicad_sch (KiCad schematic)
At the start: 2 parts, among them U1 RP2350A-QFN60, U2 VL53L4CDV0DH/1

Commit message: finished monorail
Parts:
- added C1: 100nf, symbol Device:C
- added C2: 4.7uf, symbol Device:C
- added P1: USB_C_Plug_USB2.0, symbol Connector:USB_C_Plug_USB2.0
- added R1, R2, R3, R4: 3.6k, symbol Device:R
- added R5, R6: 27K 50mW, symbol Device:R
Connections:
- net +3.3V: now also U2.11 (AVDD), C1.1, C2.1, P1.A4 (VBUS), P1.A9 (VBUS), P1.B4 (VBUS), P1.B9 (VBUS), R1.1, R2.1, R3.1, R4.1
- net GND: now also C1.2, C2.2, P1.A1 (GND), P1.A12 (GND), P1.B1 (GND), P1.B12 (GND), P1.S1 (SHIELD)
- net at U1.3 (GPIO1), U2.7 (GPIO1): now also R4.2
- net at U1.4 (GPIO2), U2.9 (SDA): now also R3.2
- net at U1.44 (ADC_AVDD): no longer U2.11 (AVDD)
- net at U1.5 (GPIO3), U2.10 (SCL): now also R2.2
- net USB_DPX: now reaches U1.51 (USB_DM)
- net USB_DPX: now also R5.1
- net USB_DMX: now reaches U1.52 (USB_DP)
- net USB_DMX: now also R6.1
- net Shutdown: now reaches U1.7 (GPIO4)
- net Shutdown: now also U2.5 (XSHUT), R1.2
- new net USB_DM: P1.A7 (D-), R6.2
- new net USB_DP: P1.A6 (D+), R5.2
- no-connect marks 1 -> 0
