File: PD Board Fused/PD Board Fused.kicad_pcb (KiCad board)
At the start: 4 copper layers, 97 x 32.5 mm, 19 parts, among them J1 Conn_02x02_Odd_Even, P1 2604-1102, P2 2604-1102, P3 2604-1102, P4 2604-1102, P5 2604-1102, P6 2604-1102, P7 2604-1102, P8 2604-1102, P9 2604-1102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

Commit message: started fused board
Parts:
- added F1: 3557-2, Customconnectors:FUSE_3557-2, F.Cu at (55.9, 88.4)
- added F2: 3557-2, Customconnectors:FUSE_3557-2, F.Cu at (55.9, 96.7)
- added F3: 3557-2, Customconnectors:FUSE_3557-2, F.Cu at (55.9, 105.0)
- added F4: 3557-2, Customconnectors:FUSE_3557-2, F.Cu at (55.9, 113.3)
- added F5: 3557-2, Customconnectors:FUSE_3557-2, F.Cu at (55.9, 121.5)
- added F6: 3557-2, Customconnectors:FUSE_3557-2, F.Cu at (55.9, 129.8)
- added F7: 3557-2, Customconnectors:FUSE_3557-2, F.Cu at (55.9, 138.1)
- added F8: 3557-2, Customconnectors:FUSE_3557-2, F.Cu at (55.9, 146.4)
Connections:
- P1 pad 3: +20V -> Net-(P1-2.1)
- P1 pad 4: +20V -> Net-(P1-2.1)
- P2 pad 3: +20V -> Net-(P2-2.1)
- P2 pad 4: +20V -> Net-(P2-2.1)
- P3 pad 3: +20V -> Net-(P3-2.1)
- P3 pad 4: +20V -> Net-(P3-2.1)
- P4 pad 3: +20V -> Net-(P4-2.1)
- P4 pad 4: +20V -> Net-(P4-2.1)
- P5 pad 3: +20V -> Net-(P5-2.1)
- P5 pad 4: +20V -> Net-(P5-2.1)
- P6 pad 3: +20V -> Net-(P6-2.1)
- P6 pad 4: +20V -> Net-(P6-2.1)
- P7 pad 3: +20V -> Net-(P7-2.1)
- P7 pad 4: +20V -> Net-(P7-2.1)
- P8 pad 3: +20V -> Net-(P8-2.1)
- P8 pad 4: +20V -> Net-(P8-2.1)

Commit message: finished monorail
Parts:
- removed J1: Conn_02x02_Odd_Even, Customconnectors:Molex_MicroFit+2x2_2068320401
- added G***: LOGO, LOGO, F.Cu at (103.2, 113.1)
- added P10: 2604-1102, Customconnectors:26041102, F.Cu at (192.1, 116.3)
- F1, F2, F3, F4, F5, F6, F7, F8: value 3557-2 -> 3544-2; footprint Customconnectors:FUSE_3557-2 -> Customconnectors:FUSE_3544-2
- moved F8 134.3 mm to (183.6, 104.7), turned to 90 degrees
- moved F4 128.0 mm to (183.6, 121.8), turned to -90 degrees
- moved F7 110.4 mm to (161.1, 104.7), turned to 90 degrees
- moved F3 106.5 mm to (161.1, 121.8), turned to -90 degrees
- moved F6 86.4 mm to (138.6, 104.7), turned to 90 degrees
- moved F2 86.4 mm to (138.6, 121.8), turned to -90 degrees
- moved F1 68.8 mm to (116.1, 121.8), turned to -90 degrees
- moved F5 62.6 mm to (116.1, 104.7), turned to 90 degrees
- moved H2 23.0 mm to (190.2, 126.7)
- moved H3 23.0 mm to (190.2, 99.8)
- moved C2 19.9 mm to (96.5, 125.3)
- moved P4 16.0 mm to (169.7, 119.4)
- moved P8 16.0 mm to (175.8, 107.1)
- moved U1 11.8 mm to (94.3, 121.9), turned to 90 degrees
- moved C1 9.96 mm to (91.2, 121.8)
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Connections:
- net Net-(P1-2.1) renamed /v1
- net Net-(P2-2.1) renamed /v2
- net Net-(P3-2.1) renamed /v3
- net Net-(P4-2.1) renamed /v4
- net Net-(P5-2.1) renamed /v5
- net Net-(P6-2.1) renamed /v6
- net Net-(P7-2.1) renamed /v7
- net Net-(P8-2.1) renamed /v8
Routing:
- net Net-(U1-VOUT): track 9.11 -> 20.4 mm
- net +20V: track 2.54 -> 0.00 mm
- net Net-(D1-A): track 3.30 -> 1.91 mm
- added copper zone on F.Cu, net /v1
- added copper zone on F.Cu, net /v2
- added copper zone on F.Cu, net /v3
- added copper zone on F.Cu, net /v4
- added copper zone on F.Cu, net /v5
- added copper zone on F.Cu, net /v6
- added copper zone on F.Cu, net /v7
- added copper zone on F.Cu, net /v8
Other:
- board size 97 x 32.5 mm -> 121.7 x 32.5 mm
- board text added: "Monorail"
