File: PD Board Fused/PD Board Fused.kicad_sch (KiCad schematic)
At the start: 19 parts, among them J1 Conn_02x02_Odd_Even, P1 2604-1102, P2 2604-1102, P3 2604-1102, P4 2604-1102, P5 2604-1102, P6 2604-1102, P7 2604-1102, P8 2604-1102, P9 2604-1102, U1 MCP1792T-3302H/CB

Commit message: started fused board
Parts:
- added F1, F2, F3, F4, F5, F6, F7, F8: 3557-2, Customconnectors:FUSE_3557-2, symbol 3557-2:3557-2
Connections:
- net +20V: now also F1.2_1, F1.2_2, F2.2_1, F2.2_2, F3.2_1, F3.2_2, F4.2_1, F4.2_2, F5.2_1, F5.2_2, F6.2_1, F6.2_2, F7.2_1, F7.2_2, F8.2_1, F8.2_2; no longer P1.3 (2.1), P1.4 (2.2), P2.3 (2.1), P2.4 (2.2), P3.3 (2.1), P3.4 (2.2), P4.3 (2.1), P4.4 (2.2), P5.3 (2.1), P5.4 (2.2), P6.3 (2.1), P6.4 (2.2), P7.3 (2.1), P7.4 (2.2), P8.3 (2.1), P8.4 (2.2)
- new net: F6.1_1, F6.1_2, P6.3 (2.1), P6.4 (2.2)
- new net: F3.1_1, F3.1_2, P3.3 (2.1), P3.4 (2.2)
- new net: F2.1_1, F2.1_2, P2.3 (2.1), P2.4 (2.2)
- new net: F5.1_1, F5.1_2, P5.3 (2.1), P5.4 (2.2)
- new net: F8.1_1, F8.1_2, P8.3 (2.1), P8.4 (2.2)
- new net: F7.1_1, F7.1_2, P7.3 (2.1), P7.4 (2.2)
- new net: F4.1_1, F4.1_2, P4.3 (2.1), P4.4 (2.2)
- new net: F1.1_1, F1.1_2, P1.3 (2.1), P1.4 (2.2)

Commit message: finished monorail
Parts:
- removed F1, F2, F3, F4, F5, F6, F7, F8: 3557-2, Customconnectors:FUSE_3557-2, symbol 3557-2:3557-2
- removed J1: Conn_02x02_Odd_Even, Customconnectors:Molex_MicroFit+2x2_2068320401, symbol Connector_Generic:Conn_02x02_Odd_Even
- added F1, F2, F3, F4, F5, F6, F7, F8: 3544-2, Customconnectors:FUSE_3544-2, symbol 3544-2:3544-2
- added P10: 2604-1102, Customconnectors:26041102, symbol 2604-1102:2604-1102
Connections:
- net +20V: now also F1.2_1, F1.2_2, F2.2_1, F2.2_2, F3.2_1, F3.2_2, F4.2_1, F4.2_2, F5.2_1, F5.2_2, F6.2_1, F6.2_2, F7.2_1, F7.2_2, F8.2_1, F8.2_2, P10.3 (2.1), P10.4 (2.2)
- net GND: now also P10.1 (1.1), P10.2 (1.2)
- net v6: now reaches P6.3 (2.1), P6.4 (2.2)
- net v6: now also F6.1_1, F6.1_2
- net v3: now reaches P3.3 (2.1), P3.4 (2.2)
- net v3: now also F3.1_1, F3.1_2
- net v2: now reaches P2.3 (2.1), P2.4 (2.2)
- net v2: now also F2.1_1, F2.1_2
- net v5: now reaches P5.3 (2.1), P5.4 (2.2)
- net v5: now also F5.1_1, F5.1_2
- net v8: now reaches P8.3 (2.1), P8.4 (2.2)
- net v8: now also F8.1_1, F8.1_2
- net v7: now reaches P7.3 (2.1), P7.4 (2.2)
- net v7: now also F7.1_1, F7.1_2
- net v4: now reaches P4.3 (2.1), P4.4 (2.2)
- net v4: now also F4.1_1, F4.1_2
- net v1: now reaches P1.3 (2.1), P1.4 (2.2)
- net v1: now also F1.1_1, F1.1_2
